File: los-fuelles.kicad_pcb (KiCad board)
At the start: 2 copper layers, 30 x 27.6 mm, 18 parts, among them J1 PWR, J2 PWR, J3 Stomp, Q1 MMBFJ201, Q2 MPSA13

Commit message: updated to KiCad 6.0
Connections:
- J3 pad 3: Net-(J3-Pad3) -> unconnected-(J3-Pad3)
